File: kicad-pcb/esp32-pedal-pcb.kicad_sch (KiCad schematic)
At the start: 28 parts, among them P1 USB_C_Plug_USB2.0, U1 MCP73871, U2 TLV75733PDBV, U3 ESP32-S3-WROOM-1

Commit message: Add BOM and update PCB design files
Parts:
- removed C1: 0.1µF, Capacitor_SMD:C_0805_2012Metric, symbol Device:C_US
- removed P1: USB_C_Plug_USB2.0, Connector_USB:USB_C_Receptacle_Palconn_UTC16-G, symbol Connector:USB_C_Plug_USB2.0
- added C1: 0.1µF, Capacitor_SMD:C_0805_2012Metric, symbol Device:C_Small_US
- added C6: 1µF, Capacitor_SMD:C_0805_2012Metric, symbol Device:C_Small_US
- added C7: 10µF, Capacitor_SMD:C_0805_2012Metric, symbol Device:C_Small_US
- added D2: SMF5V0A, Diode_SMD:D_SMF, symbol Diode:SMF5V0A
- added F1: Polyfuse_Small, Fuse:Fuse_Bourns_MF-RG500, symbol Device:Polyfuse_Small
- added J1: USB_C_Receptacle_USB2.0_14P, Connector_USB:USB_C_Receptacle_GCT_USB4110, symbol Connector:USB_C_Receptacle_USB2.0_14P
- added Q1: Q_PMOS_GSD, Package_TO_SOT_SMD:SOT-23, symbol Transistor_FET:Q_PMOS_GSD
- added R11, R12: 100kΩ, Resistor_SMD:R_0603_1608Metric, symbol Device:R_US
- added R13: 0Ω, Resistor_SMD:R_0603_1608Metric, symbol Device:R_US
- added TP6: SW1, TestPoint:TestPoint_Plated_Hole_D2.0mm, symbol Connector:TestPoint
- added TP7: SW GND, TestPoint:TestPoint_Plated_Hole_D2.0mm, symbol Connector:TestPoint
- added U4: TPD2EUSB30, Package_TO_SOT_SMD:Texas_DRT-3, symbol Power_Protection:TPD2EUSB30
- added U5: TPD2E2U06DCK, Package_TO_SOT_SMD:SOT-323_SC-70, symbol Power_Protection:TPD2E2U06DCK
- C3, C4: footprint Capacitor_SMD:C_1206_3216Metric -> Capacitor_SMD:C_0805_2012Metric
- TP1: value Rocker + -> R+
- TP2: value Rocker - -> R-
Connections:
- net GND: now also C6.1, D2.1 (A1), J1.A1 (GND), J1.A12 (GND), J1.B1 (GND), J1.B12 (GND), R11.2, R13.2, TP7.1, U4.3 (GND), U5.3
- net VBUS: now also F1.1, J1.A4 (VBUS), J1.A9 (VBUS), J1.B4 (VBUS), J1.B9 (VBUS); no longer C2.1, R5.1, U1.17 (CE)
- net at R3.1: now also J1.B5 (CC2), U5.2
- net DATA+: now reaches U3.13 (GPIO19/U1RTS/ADC2_CH8/CLK_OUT2/USB_D-)
- net DATA+: now also J1.A6 (D+), J1.B6 (D+), U4.1 (D+)
- net DATA-: now reaches U3.14 (GPIO20/U1CTS/ADC2_CH9/CLK_OUT1/USB_D+)
- net DATA-: now also J1.A7 (D-), J1.B7 (D-), U4.2 (D-)
- net at U3.23 (GPIO21): now also TP6.1
- net BOOT: now reaches Push1.2, U3.27 (GPIO0/BOOT)
- net RESET: now reaches Push2.2, U3.3 (EN)
- net RESET: now also C6.2
- net Led DIN: now reaches D1.2 (DIN), U3.38 (GPIO2/TOUCH2/ADC1_CH1)
- net at R4.1: now also J1.A5 (CC1), U5.1
- net BAT PROTECTED: now reaches TP2.1, U2.3 (EN)
- net BAT PROTECTED: now also R10.1, TP1.1, U1.14 (V_{BAT}), U1.15 (V_{BAT}), U1.16 (V_{BAT_SENSE}), Q1.2 (S)
- net at U1.2 (VPCC): now also C1.1
- new net: Q1.1 (G), R11.1, R12.1
- new net: C1.2, C7.1
- new net BAT: BT1.1 (+), Q1.3 (D), R12.2
- new net SHIELD: J1.S1 (SHIELD), R13.1
- new net VBUS PROTECTED: C2.1, C7.2, D2.2 (A2), F1.2, R5.1, U1.17 (CE)
- no-connect marks 31 -> 29
Other:
- moved on the sheet: BT1, C2, C3, C4, C5, D1, Push1, Push2, R1, R10, R2, R3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
