File: kicad-pcb/_autosave-esp32-pedal-pcb.kicad_sch (KiCad schematic)
At the start: 49 parts, among them J1 USB_C_Receptacle_USB2.0_14P, J2 Conn_01x03, J3 Conn_01x03, Q1 Q_PMOS_GSD, SW1 SW_SPST, SW2 SW_SPDT, U1 MCP73871, U2 TLV75733PDBV, U3 ESP32-S3-WROOM-1, U4 TPD2EUSB30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

Commit message: Update PCB files and documentation images
- Update KiCad PCB project files (kicad_pcb, kicad_prl, kicad_pro, kicad_sch)
- Update documentation images (3D_render.png, PCB_routing.png, schema.png)
- Add new PCB backup files
- Remove old backup files
Connections:
- net 3V3: now also R16.1, R17.1
Changed lines of the file:
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@@
+	)
+	(junction
+		(at 304.8 179.07)
+		(diameter 0)
+		(color 0 0 0 0)
 	)
 	(junction
@@
 		(color 0 0 0 0)
 	)
+	(junction
+		(at 288.29 196.85)
+		(diameter 0)
+		(color 0 0 0 0)
+	)
 	(no_connect
 		(at 243.84 190.5)
@@
 	(wire
 		(pts
+			(xy 304.8 196.85) (xy 304.8 179.07)
+		)
+		(stroke
+			(width 0)
+			(type default)
+		)
+	)
+	(wire
+		(pts
 			(xy 104.14 92.71) (xy 104.14 55.88)
 		)
@@
 		)
 		(stroke
+			(width 0)
+			(type default)
+		)
+	)
+	(wire
+		(pts
+			(xy 288.29 196.85) (xy 304.8 196.85)
+		)
+		(stroke
