File: kicad-pcb/_autosave-esp32-pedal-pcb.kicad_sch (KiCad schematic)
At the start: 54 parts, among them J1 USB4110-GF-A, SW1 B2B-PH-K-S(LF)(SN), SW2 B2B-PH-K-S(LF)(SN), U1 MCP73871T-2CCI/ML, U2 TLV75733PDBV, U3 ESP32-S3-WROOM-1-N8, U4 TPD2EUSB30ADRTR, U6 TPS2553DBVR

Commit message: Unify debug messaging across all devices using shared DebugService
- Enhanced DebugService to support both EspNowTransport (transmitters) and ReceiverEspNowTransport (receiver) via function pointers
- Migrated receiver from DebugMonitor module to shared DebugService
- Added setDeviceType() to correctly tag debug messages with device type
- Fixed grace period timing issue when clearing MAC addresses (use currentTime instead of millis())
- Improved debug messages to distinguish between no transmitters loaded vs no replies
- All devices now use the same code for sending debug messages to debug monitor
- Message buffering works consistently across all device types
Connections:
- net GPIO1: now also R20.1; no longer R15.2
- net GPIO2: now also R15.2; no longer R12.2
- net GPIO6: now also R12.2; no longer R5.1
- net GPIO7: now also R5.1; no longer R20.1
Changed lines of the file:
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@@
 		)
 	)
-	(label "GPIO7"
+	(label "GPIO1"
 		(at 213.36 227.33 0)
 		(effects
@@
 		)
 	)
-	(label "GPIO1"
+	(label "GPIO2"
 		(at 213.36 205.74 0)
 		(effects
@@
 		)
 	)
+	(label "GPIO7"
+		(at 175.26 227.33 0)
+		(effects
+			(font
+				(size 1.27 1.27)
+			)
+			(justify left bottom)
+		)
+	)
 	(label "GPIO6"
-		(at 175.26 227.33 0)
-		(effects
-			(font
-				(size 1.27 1.27)
-			)
-			(justify left bottom)
-		)
-	)
-	(label "GPIO2"
 		(at 175.26 205.74 0)
 		(effects
